File: FinalProject/Eagle/ESE350 Final Project/Column_PCB_Schematic.sch (EAGLE design)
At the start: 41 parts, among them X3 SSW-101-02-S-S

Commit message: Socket Work
Werk Werk Werk
Parts:
- removed JP1, JP2: PINHD-1X100, pinhead:PINHD-1X100
- added X4, X5, X6, X7: SSW-140-02-S-S, con-samtec:SSW-140-02-S-S
- added X8: SSW-105-02-S-S, con-samtec:SSW-105-02-S-S
- added X9: SSW-104-02-S-S, con-samtec:SSW-104-02-S-S
Connections:
- net N$100: no longer JP1.36.1
- net N$101: no longer JP1.37.1
- net N$102: no longer JP1.38.1
- net N$103: no longer JP1.39.1
- net N$104: no longer JP1.40.1
- net N$105: no longer JP1.41.1
- net N$106: no longer JP1.42.1
- net N$107: no longer JP1.43.1
- net N$108: no longer JP1.44.1
- net N$109: no longer JP1.45.1
- net N$110: no longer JP1.46.1
- net N$111: no longer JP1.47.1
- net N$112: no longer JP1.48.1
- net N$114: no longer JP1.97.1
- net N$115: no longer JP1.98.1
- net N$116: no longer JP1.99.1
- net N$117: no longer JP1.100.1
- net N$118: no longer JP2.1.1
- net N$119: no longer JP2.2.1
- net N$12: no longer JP1.1.1
- net N$120: no longer JP2.3.1
- net N$121: no longer JP2.4.1
- net N$122: no longer JP2.5.1
- net N$123: no longer JP2.6.1
- net N$124: no longer JP2.7.1
- net N$125: no longer JP2.8.1
- net N$126: no longer JP2.9.1
- net N$127: no longer JP2.10.1
- net N$128: no longer JP2.11.1
- net N$129: no longer JP2.12.1
- net N$13: no longer JP1.2.1
- net N$131: no longer JP2.13.1
- net N$132: no longer JP2.14.1
- net N$133: no longer JP2.15.1
- net N$134: no longer JP2.16.1
- net N$135: no longer JP2.17.1
- net N$136: no longer JP2.18.1
- net N$137: no longer JP2.19.1
- net N$138: no longer JP2.20.1
- net N$139: no longer JP2.21.1
- net N$14: no longer JP1.3.1
- net N$140: no longer JP2.22.1
- net N$141: no longer JP2.23.1
- net N$142: no longer JP2.24.1
- net N$143: no longer JP2.25.1
- net N$144: no longer JP2.26.1
- net N$145: no longer JP2.27.1
- net N$146: no longer JP2.28.1
- net N$148: no longer JP2.29.1
- net N$149: no longer JP2.30.1
- net N$15: no longer JP1.4.1
- net N$150: no longer JP2.31.1
- net N$151: no longer JP2.32.1
- net N$152: no longer JP2.33.1
- net N$153: no longer JP2.34.1
- net N$154: no longer JP2.35.1
- net N$155: no longer JP2.36.1
- net N$156: no longer JP2.37.1
- net N$157: no longer JP2.38.1
- net N$158: no longer JP2.39.1
- net N$159: no longer JP2.40.1
- net N$16: no longer JP1.5.1
- net N$160: no longer JP2.41.1
- net N$161: no longer JP2.42.1
- net N$162: no longer JP2.44.1
- net N$163: no longer JP2.45.1
- net N$165: no longer JP2.46.1
- net N$166: no longer JP2.47.1
- net N$167: no longer JP2.48.1
- net N$168: no longer JP2.49.1
- net N$169: no longer JP2.50.1
- net N$17: no longer JP1.6.1
- net N$170: no longer JP2.51.1
- net N$171: no longer JP2.52.1
- net N$172: no longer JP2.53.1
- net N$173: no longer JP2.54.1
- net N$174: no longer JP2.55.1
- net N$175: no longer JP2.56.1
- net N$176: no longer JP2.57.1
- net N$177: no longer JP2.58.1
- net N$178: no longer JP2.59.1
- net N$179: no longer JP2.60.1
- net N$18: no longer JP1.7.1
- net N$180: no longer JP2.61.1
- net N$182: no longer JP2.62.1
- net N$183: no longer JP2.63.1
- net N$184: no longer JP2.64.1
- net N$185: no longer JP2.65.1
- net N$186: no longer JP2.66.1
- net N$187: no longer JP2.67.1
- net N$188: no longer JP2.68.1
- net N$189: no longer JP2.69.1
- net N$19: no longer JP1.8.1
- net N$20: no longer JP1.9.1
- net N$21: no longer JP1.10.1
- net N$22: no longer JP1.11.1
- net N$23: no longer JP1.12.1
- net N$24: no longer JP1.13.1
- net N$25: no longer JP1.14.1
- net N$26: no longer JP1.15.1
- net N$27: no longer JP1.16.1
- net N$29: no longer JP1.17.1
- net N$30: no longer JP1.18.1
- net N$31: no longer JP1.19.1
- net N$32: no longer JP1.20.1
- net N$33: no longer JP1.21.1
- net N$34: no longer JP1.22.1
- net N$35: no longer JP1.23.1
- net N$36: no longer JP1.24.1
- net N$37: no longer JP1.25.1
- net N$38: no longer JP1.26.1
- net N$39: no longer JP1.27.1
- net N$40: no longer JP1.28.1
- net N$41: no longer JP1.29.1
- net N$42: no longer JP1.30.1
- net N$43: no longer JP1.31.1
- net N$44: no longer JP1.32.1
- net N$46: no longer JP1.81.1
- net N$47: no longer JP1.82.1
- net N$48: no longer JP1.83.1
- net N$49: no longer JP1.84.1
- net N$50: no longer JP1.85.1
- net N$51: no longer JP1.86.1
- net N$52: no longer JP1.87.1
- net N$53: no longer JP1.88.1
- net N$54: no longer JP1.89.1
- net N$55: no longer JP1.90.1
- net N$56: no longer JP1.91.1
- net N$57: no longer JP1.92.1
- net N$58: no longer JP1.93.1
- net N$59: no longer JP1.94.1
- net N$60: no longer JP1.95.1
- net N$61: no longer JP1.96.1
- net N$63: no longer JP1.65.1
- net N$64: no longer JP1.66.1
- net N$65: no longer JP1.67.1
- net N$66: no longer JP1.68.1
- net N$67: no longer JP1.69.1
- net N$68: no longer JP1.70.1
- net N$69: no longer JP1.71.1
- net N$70: no longer JP1.72.1
- net N$71: no longer JP1.73.1
- net N$72: no longer JP1.74.1
- net N$73: no longer JP1.75.1
- net N$74: no longer JP1.76.1
- net N$75: no longer JP1.77.1
- net N$76: no longer JP1.78.1
- net N$77: no longer JP1.79.1
- net N$78: no longer JP1.80.1
- net N$80: no longer JP1.49.1
- net N$81: no longer JP1.50.1
- net N$82: no longer JP1.51.1
- net N$83: no longer JP1.52.1
- net N$84: no longer JP1.53.1
- net N$85: no longer JP1.54.1
- net N$86: no longer JP1.55.1
- net N$87: no longer JP1.56.1
- net N$88: no longer JP1.57.1
- net N$89: no longer JP1.58.1
- net N$90: no longer JP1.59.1
- net N$91: no longer JP1.60.1
- net N$92: no longer JP1.61.1
- net N$93: no longer JP1.62.1
- net N$94: no longer JP1.63.1
- net N$95: no longer JP1.64.1
- net N$97: no longer JP1.33.1
- net N$98: no longer JP1.34.1
- net N$99: no longer JP1.35.1

Commit message: Finished Schematic
Finished hooking up the pins to the rest of the board in the schematic
and made a board. Didn’t place elements on the board, yet.
Connections:
- net N$100: now also X5-18.1
- net N$101: now also X4-19.1
- net N$102: now also X5-19.1
- net N$103: now also X4-20.1
- net N$104: now also X5-20.1
- net N$105: now also X4-21.1
- net N$106: now also X5-21.1
- net N$107: now also X4-22.1
- net N$108: now also X5-22.1
- net N$109: now also X4-23.1
- net N$110: now also X5-23.1
- net N$111: now also X4-24.1
- net N$112: now also X5-24.1
- net N$114: now also X6-9.1
- net N$115: now also X7-9.1
- net N$116: now also X6-10.1
- net N$117: now also X7-10.1
- net N$118: now also X6-11.1
- net N$119: now also X7-11.1
- net N$12: now also X4-1.1
- net N$120: now also X6-12.1
- net N$121: now also X7-12.1
- net N$122: now also X6-13.1
- net N$123: now also X7-13.1
- net N$124: now also X6-14.1
- net N$125: now also X7-14.1
- net N$126: now also X6-15.1
- net N$127: now also X7-15.1
- net N$128: now also X6-16.1
- net N$129: now also X7-16.1
- net N$13: now also X5-1.1
- net N$131: now also X6-17.1
- net N$132: now also X7-17.1
- net N$133: now also X6-18.1
- net N$134: now also X7-18.1
- net N$135: now also X6-19.1
- net N$136: now also X7-19.1
- net N$137: now also X6-20.1
- net N$138: now also X7-20.1
- net N$139: now also X6-21.1
- net N$14: now also X4-2.1
- net N$140: now also X7-21.1
- net N$141: now also X6-22.1
- net N$142: now also X7-22.1
- net N$143: now also X6-23.1
- net N$144: now also X7-23.1
- net N$145: now also X6-24.1
- net N$146: now also X7-24.1
- net N$148: now also X6-25.1
- net N$149: now also X7-25.1
- net N$15: now also X5-2.1
- net N$150: now also X6-26.1
- net N$151: now also X7-26.1
- net N$152: now also X6-27.1
- net N$153: now also X7-27.1
- net N$154: now also X6-28.1
- net N$155: now also X7-28.1
- net N$156: now also X6-29.1
- net N$157: now also X7-29.1
- net N$158: now also X6-30.1
- net N$159: now also X7-30.1
- net N$16: now also X4-3.1
- net N$160: now also X6-31.1
- net N$161: now also X7-31.1
- net N$162: now also X6-32.1
- net N$163: now also X7-32.1
- net N$165: now also X6-33.1
- net N$166: now also X7-33.1
- net N$167: now also X6-34.1
- net N$168: now also X7-34.1
- net N$169: now also X6-35.1
- net N$17: now also X5-3.1
- net N$170: now also X7-35.1
- net N$171: now also X6-36.1
- net N$172: now also X7-36.1
- net N$173: now also X6-37.1
- net N$174: now also X7-37.1
- net N$175: now also X6-38.1
- net N$176: now also X7-38.1
- net N$177: now also X6-39.1
- net N$178: now also X7-39.1
- net N$179: now also X6-40.1
- net N$18: now also X4-4.1
- net N$180: now also X7-40.1
- net N$182: now also X8-1.1
- net N$183: now also X9-1.1
- net N$184: now also X8-2.1
- net N$185: now also X9-2.1
- net N$186: now also X8-3.1
- net N$187: now also X9-3.1
- net N$188: now also X8-4.1
- net N$189: now also X9-4.1
- net N$19: now also X5-4.1
- net N$190: now also X8-5.1
- net N$20: now also X4-5.1
- net N$21: now also X5-5.1
- net N$22: now also X4-6.1
- net N$23: now also X5-6.1
- net N$24: now also X4-7.1
- net N$25: now also X5-7.1
- net N$26: now also X4-8.1
- net N$27: now also X5-8.1
- net N$29: now also X4-9.1
- net N$30: now also X5-9.1
- net N$31: now also X4-10.1
- net N$32: now also X5-10.1
- net N$33: now also X4-11.1
- net N$34: now also X5-11.1
- net N$35: now also X4-12.1
- net N$36: now also X5-12.1
- net N$37: now also X4-13.1
- net N$38: now also X5-13.1
- net N$39: now also X4-14.1
- net N$40: now also X5-14.1
- net N$41: now also X4-15.1
- net N$42: now also X5-15.1
- net N$43: now also X4-16.1
- net N$44: now also X5-16.1
- net N$46: now also X6-1.1
- net N$47: now also X7-1.1
- net N$48: now also X6-2.1
- net N$49: now also X7-2.1
- net N$50: now also X6-3.1
- net N$51: now also X7-3.1
- net N$52: now also X6-4.1
- net N$53: now also X7-4.1
- net N$54: now also X6-5.1
- net N$55: now also X7-5.1
- net N$56: now also X6-6.1
- net N$57: now also X7-6.1
- net N$58: now also X6-7.1
- net N$59: now also X7-7.1
- net N$60: now also X6-8.1
- net N$61: now also X7-8.1
- net N$63: now also X4-33.1
- net N$64: now also X5-33.1
- net N$65: now also X4-34.1
- net N$66: now also X5-34.1
- net N$67: now also X4-35.1
- net N$68: now also X5-35.1
- net N$69: now also X4-36.1
- net N$70: now also X5-36.1
- net N$71: now also X4-37.1
- net N$72: now also X5-37.1
- net N$73: now also X4-38.1
- net N$74: now also X5-38.1
- net N$75: now also X4-39.1
- net N$76: now also X5-39.1
- net N$77: now also X4-40.1
- net N$78: now also X5-40.1
- net N$80: now also X4-25.1
- net N$81: now also X5-25.1
- net N$82: now also X4-26.1
- net N$83: now also X5-26.1
- net N$84: now also X4-27.1
- net N$85: now also X5-27.1
- net N$86: now also X4-28.1
- net N$87: now also X5-28.1
- net N$88: now also X4-29.1
- net N$89: now also X5-29.1
- net N$90: now also X4-30.1
- net N$91: now also X5-30.1
- net N$92: now also X4-31.1
- net N$93: now also X5-31.1
- net N$94: now also X4-32.1
- net N$95: now also X5-32.1
- net N$97: now also X4-17.1
- net N$98: now also X5-17.1
- net N$99: now also X4-18.1
Other:
- moved on the sheet: X4-1, X4-10, X4-11, X4-12, X4-13, X4-14, X4-15, X4-16, X4-17, X4-18, X4-19, X4-2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

Commit message: Schematic Updates
Updated Schematic with modules. The schematic is now larger, and we’re
planning on having a single PCB over the back of the container.
Parts:
- removed R1, R10, R11, R12, R13, R14, R15, R16, R17, R18, R19, R2, R20, R21, R22, R23, R24, R3, R4, R5, R6, R7, R8, R9: 560K, SparkFun-Resistors:RPACK-BUSSED-8SIP-PTH-8-LP
- removed X1, X2: (no value), con-rib:SH5-5
- removed X3: SSW-101-02-S-S, con-samtec:SSW-101-02-S-S
- added C1, C10, C11, C12, C13, C2, C3, C4, C5, C6, C7, C8, C9: 0.1uF, adafruit:C-USC0402
- added IC1: 74AC11238D, 74ac-logic:74AC11238D
- added MUX_SEL: (no value), con-rib:SH5-4
- added PIN1, PIN2, PIN3, PIN4, PIN5, PIN6, PIN7: SSW-101-02-S-S, con-samtec:SSW-101-02-S-S
- added PWRSEL: (no value), con-rib:SH5-3
- added RN1: 560K, resistor-sil:G08R
- added X10, X11, X12, X13, X16, X17, X18, X19, X22, X23, X24, X25, X28, X29, X30, X31, X34, X35, X36, X37, X40, X41, X42, X43: SSW-140-02-S-S, con-samtec:SSW-140-02-S-S
- added X14, X20, X26, X32, X38, X44: SSW-105-02-S-S, con-samtec:SSW-105-02-S-S
- added X15, X21, X27, X33, X39, X45: SSW-104-02-S-S, con-samtec:SSW-104-02-S-S
Connections:
- new net BUS0: RN1.9
- new net BUS1: RN1.8
- new net BUS2: RN1.7
- new net BUS3: RN1.6
- new net BUS4: RN1.5
- new net BUS5: RN1.4
- new net BUS6: RN1.3
- new net BUS7: RN1.2
- new net N$1000: X31-13.1
- new net N$1001: X31-14.1
- new net N$1002: X31-15.1
- new net N$1003: X31-16.1
- new net N$1004: X31-17.1
- new net N$1005: X31-18.1
- new net N$1006: X31-19.1
- new net N$1007: X31-20.1
- new net N$1008: X31-21.1
- new net N$1009: X31-22.1
- new net N$1010: X31-23.1
- new net N$1011: X31-24.1
- new net N$1012: X31-25.1
- new net N$1013: X31-26.1
- new net N$1014: X31-27.1
- new net N$1015: X31-28.1
- new net N$1016: X31-29.1
- new net N$1017: X31-30.1
- new net N$1018: X31-31.1
- new net N$1019: X31-32.1
- new net N$1020: X31-33.1
- new net N$1021: X31-34.1
- new net N$1022: X31-35.1
- new net N$1023: X31-36.1
- new net N$1024: X31-37.1
- new net N$1025: X31-38.1
- new net N$1026: X31-39.1
- new net N$1027: X31-40.1
- new net N$1028: X33-1.1
- new net N$1029: X33-2.1
- new net N$1030: X33-3.1
- new net N$1031: X33-4.1
- new net N$1032: X35-1.1
- new net N$1033: X35-2.1
- new net N$1034: X35-3.1
- new net N$1035: X35-4.1
- new net N$1036: X35-5.1
- new net N$1037: X35-6.1
- new net N$1038: X35-7.1
- new net N$1039: X35-8.1
- new net N$1040: X35-9.1
- new net N$1041: X35-10.1
- new net N$1042: X35-11.1
- new net N$1043: X35-12.1
- new net N$1044: X35-13.1
- new net N$1045: X35-14.1
- new net N$1046: X35-15.1
- new net N$1047: X35-16.1
- new net N$1048: X35-17.1
- new net N$1049: X35-18.1
- new net N$1050: X35-19.1
- new net N$1051: X35-20.1
- new net N$1052: X35-21.1
- new net N$1053: X35-22.1
- new net N$1054: X35-23.1
- new net N$1055: X35-24.1
- new net N$1056: X35-25.1
- new net N$1057: X35-26.1
- new net N$1058: X35-27.1
- new net N$1059: X35-28.1
- new net N$1060: X35-29.1
- new net N$1061: X35-30.1
- new net N$1062: X35-31.1
- new net N$1063: X35-32.1
- new net N$1064: X35-33.1
- new net N$1065: X35-34.1
- new net N$1066: X35-35.1
- new net N$1067: X35-36.1
- new net N$1068: X35-37.1
- new net N$1069: X35-38.1
- new net N$1070: X35-39.1
- new net N$1071: X35-40.1
- new net N$1072: X37-1.1
- new net N$1073: X37-2.1
- new net N$1074: X37-3.1
- new net N$1075: X37-4.1
- new net N$1076: X37-5.1
- new net N$1077: X37-6.1
- new net N$1078: X37-7.1
- new net N$1079: X37-8.1
- new net N$1080: X37-9.1
- new net N$1081: X37-10.1
- new net N$1082: X37-11.1
- new net N$1083: X37-12.1
- new net N$1084: X37-13.1
- new net N$1085: X37-14.1
- new net N$1086: X37-15.1
- new net N$1087: X37-16.1
- new net N$1088: X37-17.1
- new net N$1089: X37-18.1
- new net N$1090: X37-19.1
- new net N$1091: X37-20.1
- new net N$1092: X37-21.1
- new net N$1093: X37-22.1
- new net N$1094: X37-23.1
- new net N$1095: X37-24.1
- new net N$1096: X37-25.1
- new net N$1097: X37-26.1
- new net N$1098: X37-27.1
- new net N$1099: X37-28.1
- new net N$1100: X37-29.1
- new net N$1101: X37-30.1
- new net N$1102: X37-31.1
- new net N$1103: X37-32.1
- new net N$1104: X37-33.1
- new net N$1105: X37-34.1
- new net N$1106: X37-35.1
- new net N$1107: X37-36.1
- new net N$1108: X37-37.1
- new net N$1109: X37-38.1
- new net N$1110: X37-39.1
- new net N$1111: X37-40.1
- new net N$1112: X39-1.1
- new net N$1113: X39-2.1
- new net N$1114: X39-3.1
- new net N$1115: X39-4.1
- new net N$1116: X41-1.1
- new net N$1117: X41-2.1
- new net N$1118: X41-3.1
- new net N$1119: X41-4.1
- new net N$1120: X41-5.1
- new net N$1121: X41-6.1
- new net N$1122: X41-7.1
- new net N$1123: X41-8.1
- new net N$1124: X41-9.1
- new net N$1125: X41-10.1
- new net N$1126: X41-11.1
- new net N$1127: X41-12.1
- new net N$1128: X41-13.1
- new net N$1129: X41-14.1
- new net N$1130: X41-15.1
- new net N$1131: X41-16.1
- new net N$1132: X41-17.1
- new net N$1133: X41-18.1
- new net N$1134: X41-19.1
- new net N$1135: X41-20.1
- new net N$1136: X41-21.1
- new net N$1137: X41-22.1
- new net N$1138: X41-23.1
- new net N$1139: X41-24.1
- new net N$1140: X41-25.1
- new net N$1141: X41-26.1
- new net N$1142: X41-27.1
- new net N$1143: X41-28.1
- new net N$1144: X41-29.1
- new net N$1145: X41-30.1
- new net N$1146: X41-31.1
- new net N$1147: X41-32.1
- new net N$1148: X41-33.1
- new net N$1149: X41-34.1
- new net N$1150: X41-35.1
- new net N$1151: X41-36.1
- new net N$1152: X41-37.1
- new net N$1153: X41-38.1
- new net N$1154: X41-39.1
- new net N$1155: X41-40.1
- new net N$1156: X43-1.1
- new net N$1157: X43-2.1
- new net N$1158: X43-3.1
- new net N$1159: X43-4.1
- new net N$1160: X43-5.1
- new net N$1161: X43-6.1
- new net N$1162: X43-7.1
- new net N$1163: X43-8.1
- new net N$1164: X43-9.1
- new net N$1165: X43-10.1
- new net N$1166: X43-11.1
- new net N$1167: X43-12.1
- new net N$1168: X43-13.1
- new net N$1169: X43-14.1
- new net N$1170: X43-15.1
- new net N$1171: X43-16.1
- new net N$1172: X43-17.1
- new net N$1173: X43-18.1
- new net N$1174: X43-19.1
- new net N$1175: X43-20.1
- new net N$1176: X43-21.1
- new net N$1177: X43-22.1
- new net N$1178: X43-23.1
- new net N$1179: X43-24.1
- new net N$1180: X43-25.1
- new net N$1181: X43-26.1
- new net N$1182: X43-27.1
- new net N$1183: X43-28.1
- new net N$1184: X43-29.1
- new net N$1185: X43-30.1
- new net N$1186: X43-31.1
- new net N$1187: X43-32.1
- new net N$1188: X43-33.1
- new net N$1189: X43-34.1
- new net N$1190: X43-35.1
- new net N$1191: X43-36.1
- new net N$1192: X43-37.1
- new net N$1193: X43-38.1
- new net N$1194: X43-39.1
- new net N$1195: X43-40.1
- new net N$1196: X45-1.1
- new net N$1197: X45-2.1
- new net N$1198: X45-3.1
- new net N$1199: X45-4.1
- new net N$1200: U$10.CHAN15
- new net N$1201: U$10.CHAN14
- new net N$1202: U$10.CHAN13
- new net N$1203: U$10.CHAN12
- new net N$1204: U$10.CHAN11
- new net N$1205: U$10.CHAN10
- new net N$1206: U$10.CHAN9
- new net N$1207: U$10.CHAN8
- new net N$1208: U$10.CHAN7
- new net N$1209: U$10.CHAN6
- new net N$1210: U$10.CHAN5
- new net N$1211: U$10.CHAN4
- new net N$1212: U$10.CHAN3
- new net N$1213: U$10.CHAN2
- new net N$1214: U$10.CHAN1
- new net N$1215: U$10.CHAN0
- new net N$1216: U$9.CHAN15
- new net N$1217: U$9.CHAN14
- new net N$1218: U$9.CHAN13
- new net N$1219: U$9.CHAN12
- new net N$1220: U$9.CHAN11
- new net N$1221: U$9.CHAN10
- new net N$1222: U$9.CHAN9
- new net N$1223: U$9.CHAN8
- new net N$1224: U$9.CHAN7
- new net N$1225: U$9.CHAN6
- new net N$1226: U$9.CHAN5
- new net N$1227: U$9.CHAN4
- new net N$1228: U$9.CHAN3
- new net N$1229: U$9.CHAN2
- new net N$1230: U$9.CHAN1
- new net N$1231: U$9.CHAN0
- new net N$1232: U$8.CHAN15
- new net N$1233: U$8.CHAN14
- new net N$1234: U$8.CHAN13
- new net N$1235: U$8.CHAN12
- new net N$1236: U$8.CHAN11
- new net N$1237: U$8.CHAN10
- new net N$1238: U$8.CHAN9
- new net N$1239: U$8.CHAN8
- new net N$1240: U$8.CHAN7
- new net N$1241: U$8.CHAN6
- new net N$1242: U$8.CHAN5
- new net N$1243: U$8.CHAN4
- new net N$1244: U$8.CHAN3
- new net N$1245: U$8.CHAN2
- new net N$1246: U$8.CHAN1
- new net N$1247: U$8.CHAN0
- new net N$1248: U$7.CHAN15
- new net N$1249: U$7.CHAN14
- new net N$1250: U$7.CHAN13
- new net N$1251: U$7.CHAN12
- new net N$1252: U$7.CHAN11
- new net N$1253: U$7.CHAN10
- new net N$1254: U$7.CHAN9
- new net N$1255: U$7.CHAN8
- new net N$1256: U$7.CHAN7
- new net N$1257: U$7.CHAN6
- new net N$1258: U$7.CHAN5
- new net N$1259: U$7.CHAN4
- new net N$1260: U$7.CHAN3
- new net N$1261: U$7.CHAN2
- new net N$1262: U$7.CHAN1
- new net N$1263: U$7.CHAN0
- new net N$1264: U$1.CHAN15
- new net N$1265: U$1.CHAN14
- new net N$1266: U$1.CHAN13
- new net N$1267: U$1.CHAN12
- new net N$1268: U$1.CHAN11
- new net N$1269: U$1.CHAN10
- new net N$1270: U$1.CHAN9
- new net N$1271: U$1.CHAN8
- new net N$1272: U$1.CHAN7
- new net N$1273: U$1.CHAN6
- new net N$1274: U$1.CHAN5
- new net N$1275: U$1.CHAN4
- new net N$1276: U$1.CHAN3
- new net N$1277: U$1.CHAN2
- new net N$1278: U$1.CHAN1
- new net N$1279: U$1.CHAN0
- new net N$1280: U$3.CHAN15
- new net N$1281: U$3.CHAN14
- new net N$1282: U$3.CHAN13
- new net N$1283: U$3.CHAN12
- new net N$1284: U$3.CHAN11
- new net N$1285: U$3.CHAN10
- new net N$1286: U$3.CHAN9
- new net N$1287: U$3.CHAN8
- new net N$1288: U$3.CHAN7
- new net N$1289: U$3.CHAN6
- new net N$1290: U$3.CHAN5
- new net N$1291: U$3.CHAN4
- new net N$1292: U$3.CHAN3
- new net N$1293: U$3.CHAN2
- new net N$1294: U$3.CHAN1
- new net N$1295: U$3.CHAN0
- new net N$1296: U$4.CHAN15
- new net N$1297: U$4.CHAN14
- new net N$1298: U$4.CHAN13
- new net N$1299: U$4.CHAN12
- new net N$1300: U$4.CHAN11
- new net N$1301: U$4.CHAN10
- new net N$1302: U$4.CHAN9
- new net N$1303: U$4.CHAN8
- new net N$1304: U$4.CHAN7
- new net N$1305: U$4.CHAN6
- new net N$1306: U$4.CHAN5
- new net N$1307: U$4.CHAN4
- new net N$1308: U$4.CHAN3
- new net N$1309: U$4.CHAN2
- new net N$1310: U$4.CHAN1
- new net N$1311: U$4.CHAN0
- new net N$1312: U$5.CHAN15
- new net N$1313: U$5.CHAN14
- new net N$1314: U$5.CHAN13
- new net N$1315: U$5.CHAN12
- new net N$1316: U$5.CHAN11
- new net N$1317: U$5.CHAN10
- new net N$1318: U$5.CHAN9
- new net N$1319: U$5.CHAN8
- new net N$1320: U$5.CHAN7
- new net N$1321: U$5.CHAN6
- new net N$1322: U$5.CHAN5
- new net N$1323: U$5.CHAN4
- new net N$1324: U$5.CHAN3
- new net N$1325: U$5.CHAN2
- new net N$1326: U$5.CHAN1
- new net N$1327: U$5.CHAN0
- new net N$1328: U$6.CHAN15
- new net N$1329: U$6.CHAN14
- new net N$1330: U$6.CHAN13
- new net N$1331: U$6.CHAN12
- new net N$1332: U$6.CHAN11
- new net N$1333: U$6.CHAN10
- new net N$1334: U$6.CHAN9
- new net N$1335: U$6.CHAN8
- new net N$1336: U$6.CHAN7
- new net N$1337: U$6.CHAN6
- new net N$1338: U$6.CHAN5
- new net N$1339: U$6.CHAN4
- new net N$1340: U$6.CHAN3
- new net N$1341: U$6.CHAN2
- new net N$1342: U$6.CHAN1
- new net N$1343: U$6.CHAN0
- new net N$1344: U$2.CHAN15
- new net N$1345: U$2.CHAN14
- new net N$1346: U$2.CHAN13
- new net N$1347: U$2.CHAN12
- new net N$1348: U$2.CHAN11
- new net N$1349: U$2.CHAN10
- new net N$1350: U$2.CHAN9
- new net N$1351: U$2.CHAN8
- new net N$1352: U$2.CHAN7
- new net N$1353: U$2.CHAN6
- new net N$1354: U$2.CHAN5
- new net N$1355: U$2.CHAN4
- new net N$1356: U$2.CHAN3
- new net N$1357: U$2.CHAN2
- new net N$1358: U$2.CHAN1
- new net N$1359: U$2.CHAN0
- new net N$1360: U$11.CHAN15
- new net N$1361: U$11.CHAN14
- new net N$1362: U$11.CHAN13
- new net N$1363: U$11.CHAN12
- new net N$1364: U$11.CHAN11
- new net N$1365: U$11.CHAN10
- new net N$1366: U$11.CHAN9
- new net N$1367: U$11.CHAN8
- new net N$1368: U$11.CHAN7
- new net N$1369: U$11.CHAN6
- new net N$1370: U$11.CHAN5
- new net N$1371: U$11.CHAN4
- new net N$1372: U$11.CHAN3
- new net N$1373: U$11.CHAN2
- new net N$1374: U$11.CHAN1
- new net N$1375: U$11.CHAN0
- new net N$1376: U$12.CHAN10
- new net N$1377: U$12.CHAN9
- new net N$1378: U$12.CHAN8
- new net N$1379: U$12.CHAN7
- new net N$1380: U$12.CHAN6
- new net N$1381: U$12.CHAN5
- new net N$1382: U$12.CHAN4
- new net N$1383: U$12.CHAN3
- new net N$1384: U$12.CHAN2
- new net N$1385: U$12.CHAN1
- new net N$1386: U$12.CHAN0
- new net N$1387: IC1A.A, PWRSEL-1.1
- new net N$1388: IC1A.B, PWRSEL-1.2
- new net N$1389: IC1A.C, PWRSEL-2.1
- new net N$1390: IC1A.Y0, PIN1.1, RN1.2
- new net N$1391: IC1A.Y1, PIN2.1, RN1.3
- new net N$1392: IC1A.Y2, PIN3.1, RN1.4
- new net N$1393: IC1A.Y3, PIN4.1, RN1.5
- new net N$1394: IC1A.Y4, PIN5.1, RN1.6
- new net N$1395: IC1A.Y5, PIN6.1, RN1.7
- new net N$1396: IC1A.Y6, PIN7.1, RN1.8
- new net N$1397: IC1A.Y7, RN1.9
- new net N$1398: C1.2, U$10.VCC
- new net N$1399: C2.2, U$9.VCC
- new net N$1400: C3.2, U$8.VCC
- new net N$1401: C4.2, U$7.VCC
- new net N$1402: C5.2, U$1.VCC
- new net N$1403: C6.2, U$3.VCC
- new net N$1404: C7.2, U$4.VCC
- new net N$1405: C8.2, U$5.VCC
- new net N$1406: C9.2, U$6.VCC
- new net N$1407: C10.2, U$2.VCC
- new net N$1408: C11.2, U$11.VCC
- new net N$1409: C12.2, U$12.VCC
- new net N$1410: C13.2, IC1A.G1
- new net N$198: X16-12.1
- new net N$199: X16-13.1
- new net N$200: X16-14.1
- new net N$201: X16-15.1
- new net N$202: X16-16.1
- new net N$203: X16-17.1
- new net N$204: X16-18.1
- new net N$205: X16-19.1
- new net N$206: X16-20.1
- new net N$207: X16-21.1
- new net N$208: X16-22.1
- new net N$209: X16-23.1
- new net N$210: X16-24.1
- new net N$211: X16-25.1
- new net N$212: X16-26.1
- new net N$213: X16-27.1
- new net N$214: X16-28.1
- new net N$215: X16-29.1
- new net N$216: X16-30.1
- new net N$217: X16-31.1
- new net N$218: X16-32.1
- new net N$219: X16-33.1
- new net N$220: X16-34.1
- new net N$221: X16-35.1
- new net N$222: X16-36.1
- new net N$223: X16-37.1
- new net N$224: X16-38.1
- new net N$225: X16-39.1
- new net N$226: X16-40.1
- new net N$227: X18-1.1
- new net N$228: X18-2.1
- new net N$229: X18-3.1
- new net N$230: X18-4.1
- new net N$231: X18-5.1
- new net N$232: X18-6.1
- new net N$233: X18-7.1
- new net N$234: X18-8.1
- new net N$235: X18-9.1
- new net N$236: X18-10.1
- new net N$237: X18-11.1
- new net N$238: X18-12.1
- new net N$239: X18-13.1
- new net N$240: X18-14.1
- new net N$241: X18-15.1
- new net N$242: X18-16.1
- new net N$243: X18-17.1
- new net N$244: X18-18.1
- new net N$245: X18-19.1
- new net N$246: X18-20.1
- new net N$247: X18-21.1
- new net N$248: X18-22.1
- new net N$249: X18-23.1
- new net N$250: X18-24.1
- new net N$251: X18-25.1
- new net N$252: X18-26.1
- new net N$253: X18-27.1
- new net N$254: X18-28.1
- new net N$255: X18-29.1
- new net N$256: X18-30.1
- new net N$257: X18-31.1
- new net N$258: X18-32.1
- new net N$259: X18-33.1
- new net N$260: X18-34.1
- new net N$261: X18-35.1
- new net N$262: X18-36.1
- new net N$263: X18-37.1
- new net N$264: X18-38.1
- new net N$265: X18-39.1
- new net N$266: X18-40.1
- new net N$267: X20-1.1
- new net N$268: X20-2.1
- new net N$269: X20-3.1
- new net N$270: X20-4.1
- new net N$271: X20-5.1
- new net N$272: X22-1.1
- new net N$273: X22-2.1
- new net N$274: X22-3.1
- new net N$275: X22-4.1
- new net N$276: X22-5.1
- new net N$277: X22-6.1
- new net N$278: X22-7.1
- new net N$279: X22-8.1
- new net N$28: X4-17.1
- new net N$280: X22-9.1
- new net N$281: X22-10.1
- new net N$282: X22-11.1
- new net N$283: X22-12.1
- new net N$284: X22-13.1
- new net N$285: X22-14.1
- new net N$286: X22-15.1
- new net N$287: X22-16.1
- new net N$288: X22-17.1
- new net N$289: X22-18.1
- new net N$290: X22-19.1
- new net N$291: X22-20.1
- new net N$292: X22-21.1
- new net N$293: X22-22.1
- new net N$294: X22-23.1
- new net N$295: X22-24.1
- new net N$296: X22-25.1
- new net N$297: X22-26.1
- new net N$298: X22-27.1
- new net N$299: X22-28.1
- new net N$300: X22-29.1
- new net N$301: X22-30.1
- new net N$302: X22-31.1
- new net N$303: X22-32.1
- new net N$304: X22-33.1
- new net N$305: X22-34.1
- new net N$306: X22-35.1
- new net N$307: X22-36.1
- new net N$308: X22-37.1
- new net N$309: X22-38.1
- new net N$310: X22-39.1
- new net N$311: X22-40.1
- new net N$312: X24-1.1
- new net N$313: X24-2.1
- new net N$314: X24-3.1
- new net N$315: X24-4.1
- new net N$316: X24-5.1
- new net N$317: X24-6.1
- new net N$318: X24-7.1
- new net N$319: X24-8.1
- new net N$320: X24-9.1
- new net N$321: X24-10.1
- new net N$322: X24-11.1
- new net N$323: X24-12.1
- new net N$324: X24-13.1
- new net N$325: X24-14.1
- new net N$326: X24-15.1
- new net N$327: X24-16.1
- new net N$328: X24-17.1
- new net N$329: X24-18.1
- new net N$330: X24-19.1
- new net N$331: X24-20.1
- new net N$332: X24-21.1
- new net N$333: X24-22.1
- new net N$334: X24-23.1
- new net N$335: X24-24.1
- new net N$336: X24-25.1
- new net N$337: X24-26.1
- new net N$338: X24-27.1
- new net N$339: X24-28.1
- new net N$340: X24-29.1
- new net N$341: X24-30.1
- new net N$342: X24-31.1
- new net N$343: X24-32.1
- new net N$344: X24-33.1
- new net N$345: X24-34.1
- new net N$346: X24-35.1
- new net N$347: X24-36.1
- new net N$348: X24-37.1
- new net N$349: X24-38.1
- new net N$350: X24-39.1
- new net N$351: X24-40.1
- new net N$352: X26-1.1
- new net N$353: X26-2.1
- new net N$354: X26-3.1
- new net N$355: X26-4.1
- new net N$356: X26-5.1
- new net N$357: X28-1.1
- new net N$358: X28-2.1
- new net N$359: X28-3.1
- new net N$360: X28-4.1
- new net N$361: X28-5.1
- new net N$362: X28-6.1
- new net N$363: X28-7.1
- new net N$364: X28-8.1
- new net N$365: X28-9.1
- new net N$366: X28-10.1
- new net N$367: X28-11.1
- new net N$368: X28-12.1
- new net N$369: X28-13.1
- new net N$370: X28-14.1
- new net N$371: X28-15.1
- new net N$372: X28-16.1
- new net N$373: X28-17.1
- new net N$374: X28-18.1
- new net N$375: X28-19.1
- new net N$376: X28-20.1
- new net N$377: X28-21.1
- new net N$378: X28-22.1
- new net N$379: X28-23.1
- new net N$380: X28-24.1
- new net N$381: X28-25.1
- new net N$382: X28-26.1
- new net N$383: X28-27.1
- new net N$384: X28-28.1
- new net N$385: X28-29.1
- new net N$386: X28-30.1
- new net N$387: X28-31.1
- new net N$388: X28-32.1
- new net N$389: X28-33.1
- new net N$390: X28-34.1
- new net N$391: X28-35.1
- new net N$392: X28-36.1
- new net N$393: X28-37.1
- new net N$394: X28-38.1
- new net N$395: X28-39.1
- new net N$396: X28-40.1
- new net N$397: X30-1.1
- new net N$398: X30-2.1
- new net N$399: X30-3.1
- new net N$400: X30-4.1
- new net N$401: X30-5.1
- new net N$402: X30-6.1
- new net N$403: X30-7.1
- new net N$404: X30-8.1
- new net N$405: X30-9.1
- new net N$406: X30-10.1
- new net N$407: X30-11.1
- new net N$408: X30-12.1
- new net N$409: X30-13.1
- new net N$410: X30-14.1
- new net N$411: X30-15.1
- new net N$412: X30-16.1
- new net N$413: X30-17.1
- new net N$414: X30-18.1
- new net N$415: X30-19.1
- new net N$416: X30-20.1
- new net N$417: X30-21.1
- new net N$418: X30-22.1
- new net N$419: X30-23.1
- new net N$420: X30-24.1
- new net N$421: X30-25.1
- new net N$422: X30-26.1
- new net N$423: X30-27.1
- new net N$424: X30-28.1
- new net N$425: X30-29.1
- new net N$426: X30-30.1
- new net N$427: X30-31.1
- new net N$428: X30-32.1
- new net N$429: X30-33.1
- new net N$430: X30-34.1
- new net N$431: X30-35.1
- new net N$432: X30-36.1
- new net N$433: X30-37.1
- new net N$434: X30-38.1
- new net N$435: X30-39.1
- new net N$436: X30-40.1
- new net N$437: X32-1.1
- new net N$438: X32-2.1
- new net N$439: X32-3.1
- new net N$440: X32-4.1
- new net N$441: X32-5.1
- new net N$442: X34-1.1
- new net N$443: X34-2.1
- new net N$444: X34-3.1
- new net N$445: X34-4.1
- new net N$446: X34-5.1
- new net N$447: X34-6.1
- new net N$448: X34-7.1
- new net N$449: X34-8.1
- new net N$45: X4-34.1
- new net N$450: X34-9.1
- new net N$451: X34-10.1
- new net N$452: X34-11.1
- new net N$453: X34-12.1
- new net N$454: X34-13.1
- new net N$455: X34-14.1
- new net N$456: X34-15.1
- new net N$457: X34-16.1
- new net N$458: X34-17.1
- new net N$459: X34-18.1
- new net N$460: X34-19.1
- new net N$461: X34-20.1
- new net N$462: X34-21.1
- new net N$463: X34-22.1
- new net N$464: X34-23.1
- new net N$465: X34-24.1
- new net N$466: X34-25.1
- new net N$467: X34-26.1
- new net N$468: X34-27.1
- new net N$469: X34-28.1
- new net N$470: X34-29.1
- new net N$471: X34-30.1
- new net N$472: X34-31.1
- new net N$473: X34-32.1
- new net N$474: X34-33.1
- new net N$475: X34-34.1
- new net N$476: X34-35.1
- new net N$477: X34-36.1
- new net N$478: X34-37.1
- new net N$479: X34-38.1
- new net N$480: X34-39.1
- new net N$481: X34-40.1
- new net N$482: X36-1.1
- new net N$483: X36-2.1
- new net N$484: X36-3.1
- new net N$485: X36-4.1
- new net N$486: X36-5.1
- new net N$487: X36-6.1
- new net N$488: X36-7.1
- new net N$489: X36-8.1
- new net N$490: X36-9.1
- new net N$491: X36-10.1
- new net N$492: X36-11.1
- new net N$493: X36-12.1
- new net N$494: X36-13.1
- new net N$495: X36-14.1
- new net N$496: X36-15.1
- new net N$497: X36-16.1
- new net N$498: X36-17.1
- new net N$499: X36-18.1
- new net N$500: X36-19.1
- new net N$501: X36-20.1
- new net N$502: X36-21.1
- new net N$503: X36-22.1
- new net N$504: X36-23.1
- new net N$505: X36-24.1
- new net N$506: X36-25.1
- new net N$507: X36-26.1
- new net N$508: X36-27.1
- new net N$509: X36-28.1
- new net N$510: X36-29.1
- new net N$511: X36-30.1
- new net N$512: X36-31.1
- new net N$513: X36-32.1
- new net N$514: X36-33.1
- new net N$515: X36-34.1
- new net N$516: X36-35.1
- new net N$517: X36-36.1
- new net N$518: X36-37.1
- new net N$519: X36-38.1
- new net N$520: X36-39.1
- new net N$521: X36-40.1
- new net N$522: X38-1.1
- new net N$523: X38-2.1
- new net N$524: X38-3.1
- new net N$525: X38-4.1
- new net N$526: X38-5.1
- new net N$527: X40-1.1
- new net N$528: X40-2.1
- new net N$529: X40-3.1
- new net N$530: X40-4.1
- new net N$531: X40-5.1
- new net N$532: X40-6.1
- new net N$533: X40-7.1
- new net N$534: X40-8.1
- new net N$535: X40-9.1
- new net N$536: X40-10.1
- new net N$537: X40-11.1
- new net N$538: X40-12.1
- new net N$539: X40-13.1
- new net N$540: X40-14.1
- new net N$541: X40-15.1
- new net N$542: X40-16.1
- new net N$543: X40-17.1
- new net N$544: X40-18.1
- new net N$545: X40-19.1
- new net N$546: X40-20.1
- new net N$547: X40-21.1
- new net N$548: X40-22.1
- new net N$549: X40-23.1
- new net N$550: X40-24.1
- new net N$551: X40-25.1
- new net N$552: X40-26.1
- new net N$553: X40-27.1
- new net N$554: X40-28.1
- new net N$555: X40-29.1
- new net N$556: X40-30.1
- new net N$557: X40-31.1
- new net N$558: X40-32.1
- new net N$559: X40-33.1
- new net N$560: X40-34.1
- new net N$561: X40-35.1
- new net N$562: X40-36.1
- new net N$563: X40-37.1
- new net N$564: X40-38.1
- new net N$565: X40-39.1
- new net N$566: X40-40.1
- new net N$567: X42-1.1
- new net N$568: X42-2.1
- new net N$569: X42-3.1
- new net N$570: X42-4.1
- new net N$571: X42-5.1
- new net N$572: X42-6.1
- new net N$573: X42-7.1
- new net N$574: X42-8.1
- new net N$575: X42-9.1
- new net N$576: X42-10.1
- new net N$577: X42-11.1
- new net N$578: X42-12.1
- new net N$579: X42-13.1
- new net N$580: X42-14.1
- new net N$581: X42-15.1
- new net N$582: X42-16.1
- new net N$583: X42-17.1
- new net N$584: X42-18.1
- new net N$585: X42-19.1
- new net N$586: X42-20.1
- new net N$587: X42-21.1
- new net N$588: X42-22.1
- new net N$589: X42-23.1
- new net N$590: X42-24.1
- new net N$591: X42-25.1
- new net N$592: X42-26.1
- new net N$593: X42-27.1
- new net N$594: X42-28.1
- new net N$595: X42-29.1
- new net N$596: X42-30.1
- new net N$597: X42-31.1
- new net N$598: X42-32.1
- new net N$599: X42-33.1
- new net N$600: X42-34.1
- new net N$601: X42-35.1
- new net N$602: X42-36.1
- new net N$603: X42-37.1
- new net N$604: X42-38.1
- new net N$605: X42-39.1
- new net N$606: X42-40.1
- new net N$607: X44-1.1
- new net N$608: X44-2.1
- new net N$609: X44-3.1
- new net N$610: X44-4.1
- new net N$611: X44-5.1
- new net N$612: X5-1.1
- new net N$613: X5-2.1
- new net N$614: X5-3.1
- new net N$615: X5-4.1
- new net N$616: X5-5.1
- new net N$617: X5-6.1
- new net N$618: X5-7.1
- new net N$619: X5-8.1
- new net N$62: X6-11.1
- new net N$620: X5-9.1
- new net N$621: X5-10.1
- new net N$622: X5-11.1
- new net N$623: X5-12.1
- new net N$624: X5-13.1
- new net N$625: X5-14.1
- new net N$626: X5-15.1
- new net N$627: X5-16.1
- new net N$628: X5-17.1
- new net N$629: X5-18.1
- new net N$630: X5-19.1
- new net N$631: X5-20.1
- new net N$632: X5-21.1
- new net N$633: X5-22.1
- new net N$634: X5-23.1
- new net N$635: X5-24.1
- new net N$636: X5-25.1
- new net N$637: X5-26.1
- new net N$638: X5-27.1
- new net N$639: X5-28.1
- new net N$640: X5-29.1
- new net N$641: X5-30.1
- new net N$642: X5-31.1
- new net N$643: X5-32.1
- new net N$644: X5-33.1
- new net N$645: X5-34.1
- new net N$646: X5-35.1
- new net N$647: X5-36.1
- new net N$648: X5-37.1
- new net N$649: X5-38.1
- new net N$650: X5-39.1
- new net N$651: X5-40.1
- new net N$652: X7-1.1
- new net N$653: X7-2.1
- new net N$654: X7-3.1
- new net N$655: X7-4.1
- new net N$656: X7-5.1
- new net N$657: X7-6.1
- new net N$658: X7-7.1
- new net N$659: X7-8.1
- new net N$660: X7-9.1
- new net N$661: X7-10.1
- new net N$662: X7-11.1
- new net N$663: X7-12.1
- new net N$664: X7-13.1
- new net N$665: X7-14.1
- new net N$666: X7-15.1
- new net N$667: X7-16.1
- new net N$668: X7-17.1
- new net N$669: X7-18.1
- new net N$670: X7-19.1
- new net N$671: X7-20.1
- new net N$672: X7-21.1
- new net N$673: X7-22.1
- new net N$674: X7-23.1
- new net N$675: X7-24.1
- new net N$676: X7-25.1
- new net N$677: X7-26.1
- new net N$678: X7-27.1
- new net N$679: X7-28.1
- new net N$680: X7-29.1
- new net N$681: X7-30.1
- new net N$682: X7-31.1
- new net N$683: X7-32.1
- new net N$684: X7-33.1
- new net N$685: X7-34.1
- new net N$686: X7-35.1
- new net N$687: X7-36.1
- new net N$688: X7-37.1
- new net N$689: X7-38.1
- new net N$690: X7-39.1
- new net N$691: X7-40.1
- new net N$692: X9-1.1
- new net N$693: X9-2.1
- new net N$694: X9-3.1
- new net N$695: X9-4.1
- new net N$696: X11-1.1
- new net N$697: X11-2.1
- new net N$698: X11-3.1
- new net N$699: X11-4.1
- new net N$700: X11-5.1
- new net N$701: X11-6.1
- new net N$702: X11-7.1
- new net N$703: X11-8.1
- new net N$704: X11-9.1
- new net N$705: X11-10.1
- new net N$706: X11-11.1
- new net N$707: X11-12.1
- new net N$708: X11-13.1
- new net N$709: X11-14.1
- new net N$710: X11-15.1
- new net N$711: X11-16.1
- new net N$712: X11-17.1
- new net N$713: X11-18.1
- new net N$714: X11-19.1
- new net N$715: X11-20.1
- new net N$716: X11-21.1
- new net N$717: X11-22.1
- new net N$718: X11-23.1
- new net N$719: X11-24.1
- new net N$720: X11-25.1
- new net N$721: X11-26.1
- new net N$722: X11-27.1
- new net N$723: X11-28.1
- new net N$724: X11-29.1
- new net N$725: X11-30.1
- new net N$726: X11-31.1
- new net N$727: X11-32.1
- new net N$728: X11-33.1
- new net N$729: X11-34.1
- new net N$730: X11-35.1
- new net N$731: X11-36.1
- new net N$732: X11-37.1
- new net N$733: X11-38.1
- new net N$734: X11-39.1
- new net N$735: X11-40.1
- new net N$736: X13-1.1
- new net N$737: X13-2.1
- new net N$738: X13-3.1
- new net N$739: X13-4.1
- new net N$740: X13-5.1
- new net N$741: X13-6.1
- new net N$742: X13-7.1
- new net N$743: X13-8.1
- new net N$744: X13-9.1
- new net N$745: X13-10.1
- new net N$746: X13-11.1
- new net N$747: X13-12.1
- new net N$748: X13-13.1
- new net N$749: X13-14.1
- new net N$750: X13-15.1
- new net N$751: X13-16.1
- new net N$752: X13-17.1
- new net N$753: X13-18.1
- new net N$754: X13-19.1
- new net N$755: X13-20.1
- new net N$756: X13-21.1
- new net N$757: X13-22.1
- new net N$758: X13-23.1
- new net N$759: X13-24.1
- new net N$760: X13-25.1
- new net N$761: X13-26.1
- new net N$762: X13-27.1
- new net N$763: X13-28.1
- new net N$764: X13-29.1
- new net N$765: X13-30.1
- new net N$766: X13-31.1
- new net N$767: X13-32.1
- new net N$768: X13-33.1
- new net N$769: X13-34.1
- new net N$770: X13-35.1
- new net N$771: X13-36.1
- new net N$772: X13-37.1
- new net N$773: X13-38.1
- new net N$774: X13-39.1
- new net N$775: X13-40.1
- new net N$776: X15-1.1
- new net N$777: X15-2.1
- new net N$778: X15-3.1
- new net N$779: X15-4.1
- new net N$780: X17-1.1
- new net N$781: X17-2.1
- new net N$782: X17-3.1
- new net N$783: X17-4.1
- new net N$784: X17-5.1
- new net N$785: X17-6.1
- new net N$786: X17-7.1
- new net N$787: X17-8.1
- new net N$788: X17-9.1
- new net N$789: X17-10.1
- new net N$79: X6-28.1
- new net N$790: X17-11.1
- new net N$791: X17-12.1
- new net N$792: X17-13.1
- new net N$793: X17-14.1
- new net N$794: X17-15.1
- new net N$795: X17-16.1
- new net N$796: X17-17.1
- new net N$797: X17-18.1
- new net N$798: X17-19.1
- new net N$799: X17-20.1
- new net N$800: X17-21.1
- new net N$801: X17-22.1
- new net N$802: X17-23.1
- new net N$803: X17-24.1
- new net N$804: X17-25.1
- new net N$805: X17-26.1
- new net N$806: X17-27.1
- new net N$807: X17-28.1
- new net N$808: X17-29.1
- new net N$809: X17-30.1
- new net N$810: X17-31.1
- new net N$811: X17-32.1
- new net N$812: X17-33.1
- new net N$813: X17-34.1
- new net N$814: X17-35.1
- new net N$815: X17-36.1
- new net N$816: X17-37.1
- new net N$817: X17-38.1
- new net N$818: X17-39.1
- new net N$819: X17-40.1
- new net N$820: X19-1.1
- new net N$821: X19-2.1
- new net N$822: X19-3.1
- new net N$823: X19-4.1
- new net N$824: X19-5.1
- new net N$825: X19-6.1
- new net N$826: X19-7.1
- new net N$827: X19-8.1
- new net N$828: X19-9.1
- new net N$829: X19-10.1
- new net N$830: X19-11.1
- new net N$831: X19-12.1
- new net N$832: X19-13.1
- new net N$833: X19-14.1
- new net N$834: X19-15.1
- new net N$835: X19-16.1
- new net N$836: X19-17.1
- new net N$837: X19-18.1
- new net N$838: X19-19.1
- new net N$839: X19-20.1
- new net N$840: X19-21.1
- new net N$841: X19-22.1
- new net N$842: X19-23.1
- new net N$843: X19-24.1
- new net N$844: X19-25.1
- new net N$845: X19-26.1
- new net N$846: X19-27.1
- new net N$847: X19-28.1
- new net N$848: X19-29.1
- new net N$849: X19-30.1
- new net N$850: X19-31.1
- new net N$851: X19-32.1
- new net N$852: X19-33.1
- new net N$853: X19-34.1
- new net N$854: X19-35.1
- new net N$855: X19-36.1
- new net N$856: X19-37.1
- new net N$857: X19-38.1
- new net N$858: X19-39.1
- new net N$859: X19-40.1
- new net N$860: X21-1.1
- new net N$861: X21-2.1
- new net N$862: X21-3.1
- new net N$863: X21-4.1
- new net N$864: X23-1.1
- new net N$865: X23-2.1
- new net N$866: X23-3.1
- new net N$867: X23-4.1
- new net N$868: X23-5.1
- new net N$869: X23-6.1
- new net N$870: X23-7.1
- new net N$871: X23-8.1
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Other:
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